File: cr2-clone/MCU.kicad_sch (KiCad schematic)
At the start: 21 parts, among them U2 nRF52840, Y1 32Mhz

Commit message: added power block
Parts:
- removed L4: L, symbol Device:L
- removed L5: 10uH, symbol Device:L
- added C20, C21: C, symbol Device:C
- added D2: LED, LED_SMD:LED_0805_2012Metric_Pad1.15x1.40mm_HandSolder, symbol Device:LED
- added D3, D4: LED, symbol Device:LED
- added R3, R4, R5: 330, Resistor_SMD:R_0805_2012Metric_Pad1.20x1.40mm_HandSolder, symbol Device:R
- added SW1: Boot, Button_Switch_SMD:SW_MEC_5GSH9, symbol Switch:SW_Push
- added SW2: Reset, symbol Switch:SW_Push
- C10: value 100pF -> NC
- C11: value 100nF -> 100pF
- C13: value NC -> 100nF
- L3: value L -> 4n7
Connections:
- net +5V: no longer U2.Y2 (VDDH)
- net DEC: no longer L3.2
- net GND: now also C20.1, C21.2, D2.1 (K), D3.1 (K), D4.1 (K), SW1.2, SW2.2
- net VCC: now also U2.Y2 (VDDH)
- net DEC1: now reaches U2.C1 (DEC1)
- net DEC1: now also C13.2; no longer C11.2
- net DEC5: now reaches U2.N24 (DEC5)
- net DEC5: now also C10.2; no longer C13.2
- net DEC2: now reaches C12.2, U2.A18 (DEC2)
- net Reset: now reaches J2.4 (Pin_4), U2.AC13 (P0.18/~{RESET})
- net Reset: now also SW2.1
- net DECUSB: now reaches C5.2, U2.AC5 (DECUSB)
- net LED_R: now reaches U2.AD16 (P0.20)
- net LED_R: now also R3.1
- net LED_G: now reaches U2.AD18 (P0.22)
- net LED_G: now also R4.1
- net LED_B: now reaches U2.AD20 (P0.24)
- net LED_B: now also R5.1
- net Boot: now reaches U2.D2 (XL1/P0.00)
- net Boot: now also SW1.1
- net DEC3: now reaches U2.D23 (DEC3)
- net DEC3: now also C11.2; no longer C10.2
- net at U2.H23 (ANT): now also L3.2, C20.2
- net ANT: now reaches L3.1
- net ANT: now also C21.1
- new net: D4.2 (A), R5.2
- new net: D2.2 (A), R3.2
- new net: D3.2 (A), R4.2
- no-connect marks 0 -> 2

Commit message: added peripherals
Parts:
- removed J2: ~, Connector_Molex:Molex_KK-254_AE-6410-05A_1x05_P2.54mm_Vertical, symbol Connector_Generic:Conn_01x05
- added J3: Conn_01x04, Connector_JST:JST_EH_B4B-EH-A_1x04_P2.50mm_Vertical, symbol Connector_Generic:Conn_01x04
- added J4: Conn_01x03, Connector_JST:JST_EH_B3B-EH-A_1x03_P2.50mm_Vertical, symbol Connector_Generic:Conn_01x03
- added J5: Conn_01x06, Connector_JST:JST_EH_B6B-EH-A_1x06_P2.50mm_Vertical, symbol Connector_Generic:Conn_01x06
- added L4: 10u, symbol Device:L
- added L5: 15nH, symbol Device:L
Connections:
- net +5V: now also J3.1 (Pin_1), J5.6 (Pin_6)
- net DEC: now also L5.2
- net GND: now also U2.A10 (AIN5/P0.29), U2.B9 (AIN6/P0.30), J3.4 (Pin_4), J4.3 (Pin_3), J5.4 (Pin_4)
- net Reset: now also U2.AD12 (P0.17), J5.2 (Pin_2)
- net VCC: now also J3.2 (Pin_2)
- net RX_EN: now reaches U2.A14 (P1.15)
- net PA_ANT_SEL: now reaches U2.A16 (P1.13)
- net TX_EN: now reaches U2.A20 (P1.10)
- net PA_MODE: now reaches U2.A8 (AIN7/P0.31)
- net SWDCLK: now reaches U2.AA24 (SWDCLK)
- net SWDCLK: now also J5.5 (Pin_5)
- net SWDIO: now reaches U2.AC24 (SWDIO)
- net SWDIO: now also J5.3 (Pin_3)
- net SWO: now reaches U2.AD22 (TRACEDATA0/P1.00)
- net SWO: now also J5.1 (Pin_1)
- net at U2.B3 (DCC): now also L4.1
- net IO2: now reaches U2.G1 (P0.26)
- net IO2: now also J4.1 (Pin_1)
- net IO1: now reaches U2.J1 (AIN2/P0.04)
- net IO1: now also J4.2 (Pin_2)
- net PA_PDN: now reaches U2.J24 (NFC2/P0.10)
- net PA_SCK: now reaches U2.L24 (NFC1/P0.09)
- net IO3: now reaches U2.N1 (P0.08)
- net IO3: now also J3.3 (Pin_3)
- net PA_SDO: now reaches U2.R24 (P1.06)
- net PA_SDI: now reaches U2.U24 (P1.04)
- net PA_CS: now reaches U2.W24 (P1.02)
- net D+ renamed D_P
- net D- renamed D_N
- new net: L4.2, L5.1
- no-connect marks 2 -> 30

Commit message: added footprint, init pcb design
Parts:
- C10, C11, C12, C13, C14, C15, C16, C17, C18, C19, C20, C21, C5, C6, C7, C8, C9: footprint (none) -> Capacitor_SMD:C_0603_1608Metric_Pad1.08x0.95mm_HandSolder
- D2: footprint LED_SMD:LED_0805_2012Metric_Pad1.15x1.40mm_HandSolder -> LED_SMD:LED_0603_1608Metric_Pad1.05x0.95mm_HandSolder
- D3, D4: footprint (none) -> LED_SMD:LED_0603_1608Metric_Pad1.05x0.95mm_HandSolder
- L3, L4, L5: footprint (none) -> Inductor_SMD:L_0603_1608Metric_Pad1.05x0.95mm_HandSolder
- R3, R4, R5: footprint Resistor_SMD:R_0805_2012Metric_Pad1.20x1.40mm_HandSolder -> Resistor_SMD:R_0603_1608Metric_Pad0.98x0.95mm_HandSolder
- SW1: footprint Button_Switch_SMD:SW_MEC_5GSH9 -> Button_Switch_SMD:SW_Push_1P1T_NO_6x6mm_H9.5mm
- SW2: footprint (none) -> Button_Switch_SMD:SW_Push_1P1T_NO_6x6mm_H9.5mm
Connections:
- no-connect marks 30 -> 28
Changed lines of the file:
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@@
 (kicad_sch (version 20230121) (generator eeschema)
   (paper "A4")
+  (junction (at 116.84 187.96) (diameter 0) (color 0 0 0 0)
+  )
   (junction (at 228.6 90.17) (diameter 0) (color 0 0 0 0)
   )
@@
   (junction (at 168.91 24.13) (diameter 0) (color 0 0 0 0)
   )
-  (junction (at 114.3 187.96) (diameter 0) (color 0 0 0 0)
-  )
   (junction (at 223.52 90.17) (diameter 0) (color 0 0 0 0)
   )
@@
   (junction (at 200.66 27.94) (diameter 0) (color 0 0 0 0)
   )
-  (no_connect (at 142.24 52.07))
   (no_connect (at 147.32 57.15))
   (no_connect (at 147.32 67.31))
@@
   (no_connect (at 147.32 120.65))
   (no_connect (at 147.32 135.89))
-  (no_connect (at 148.59 64.77))
   (no_connect (at 147.32 118.11))
   (no_connect (at 147.32 85.09))
@@
     (stroke (width 0) (type default))
   )
-  (wire (pts (xy 114.3 187.96) (xy 114.3 189.23))
+  (wire (pts (xy 116.84 187.96) (xy 116.84 190.5))
     (stroke (width 0) (type default))
   )
@@
       (effects (font (size 1.27 1.27)))
     )
-    (property "Footprint" "" (at 189.23 153.67 0)
+    (property "Footprint" "LED_SMD:LED_0603_1608Metric_Pad1.05x0.95mm_HandSolder" (at 189.23 153.67 0)
       (effects (font (size 1.27 1.27)) hide)
     )
@@
       (effects (font (size 1.27 1.27)))
     )
-    (property "Footprint" "" (at 69.85 109.5248 0)
+    (property "Footprint" "Capacitor_SMD:C_0603_1608Metric_Pad1.08x0.95mm_HandSolder" (at 69.85 109.5248 0)
       (effects (font (size 1.27 1.27)) hide)
     )
@@
       (effects (font (size 1.27 1.27)))
     )
-    (property "Footprint" "" (at 62.23 121.6152 0)
+    (property "Footprint" "Capacitor_SMD:C_0603_1608Metric_Pad1.08x0.95mm_HandSolder" (at 62.23 121.6152 0)
       (effects (font (size 1.27 1.27)) hide)
     )
@@
       (effects (font (size 1.27 1.27)) (justify left))
     )
-    (property "Footprint" "" (at 63.1952 77.47 0)
+    (property "Footprint" "Capacitor_SMD:C_0603_1608Metric_Pad1.08x0.95mm_HandSolder" (at 63.1952 77.47 0)
       (effects (font (size 1.27 1.27)) hide)
     )
@@
       (effects (font (size 1.27 1.27)) (justify left))
     )
-    (property "Footprint" "" (at 180.0352 24.13 0)
+    (property "Footprint" "Capacitor_SMD:C_0603_1608Metric_Pad1.08x0.95mm_HandSolder" (at 180.0352 24.13 0)
       (effects (font (size 1.27 1.27)) hide)
     )
@@
       (effects (font (size 1.27 1.27)))
     )
-    (property "Footprint" "" (at 147.32 30.48 0)
+    (property "Footprint" "Inductor_SMD:L_0603_1608Metric_Pad1.05x0.95mm_HandSolder" (at 147.32 30.48 0)
       (effects (font (size 1.27 1.27)) hide)
     )
@@
       (effects (font (size 1.27 1.27)))
     )
-    (property "Footprint" "LED_SMD:LED_0805_2012Metric_Pad1.15x1.40mm_HandSolder" (at 189.23 139.7 0)
+    (property "Footprint" "LED_SMD:LED_0603_1608Metric_Pad1.05x0.95mm_HandSolder" (at 189.23 139.7 0)
       (effects (font (size 1.27 1.27)) hide)
     )
@@
       (effects (font (size 1.27 1.27)) (justify left))
     )
-    (property "Footprint" "" (at 223.2152 26.67 0)
+    (property "Footprint" "Capacitor_SMD:C_0603_1608Metric_Pad1.08x0.95mm_HandSolder" (at 223.2152 26.67 0)
       (effects (font (size 1.27 1.27)) hide)
     )
@@
       (effects (font (size 1.27 1.27)) (justify left))
     )
-    (property "Footprint" "" (at 222.5548 82.55 0)
+    (property "Footprint" "Capacitor_SMD:C_0603_1608Metric_Pad1.08x0.95mm_HandSolder" (at 222.5548 82.55 0)
       (effects (font (size 1.27 1.27)) hide)
     )
@@
       (effects (font (size 1.27 1.27)))
     )
-    (property "Footprint" "" (at 189.23 146.05 0)
+    (property "Footprint" "LED_SMD:LED_0603_1608Metric_Pad1.05x0.95mm_HandSolder" (at 189.23 146.05 0)
       (effects (font (size 1.27 1.27)) hide)
     )
@@
       (effects (font (size 1.27 1.27)) (justify left))
     )
-    (property "Footprint" "" (at 213.6648 82.55 0)
+    (property "Footprint" "Capacitor_SMD:C_0603_1608Metric_Pad1.08x0.95mm_HandSolder" (at 213.6648 82.55 0)
       (effects (font (size 1.27 1.27)) hide)
     )
@@
       (effects (font (size 1.27 1.27)))
     )
-    (property "Footprint" "" (at 138.43 30.48 0)
+    (property "Footprint" "Inductor_SMD:L_0603_1608Metric_Pad1.05x0.95mm_HandSolder" (at 138.43 30.48 0)
       (effects (font (size 1.27 1.27)) hide)
     )
@@
       (effects (font (size 1.27 1.27)))
     )
-    (property "Footprint" "Resistor_SMD:R_0805_2012Metric_Pad1.20x1.40mm_HandSolder" (at 181.61 155.448 90)
+    (property "Footprint" "Resistor_SMD:R_0603_1608Metric_Pad0.98x0.95mm_HandSolder" (at 181.61 155.448 90)
       (effects (font (size 1.27 1.27)) hide)
     )
@@
       (effects (font (size 1.27 1.27)) (justify left))
     )
-    (property "Footprint" "" (at 233.9848 82.55 0)
+    (property "Footprint" "Capacitor_SMD:C_0603_1608Metric_Pad1.08x0.95mm_HandSolder" (at 233.9848 82.55 0)
       (effects (font (size 1.27 1.27)) hide)
     )
@@
       (effects (font (size 1.27 1.27)))
     )
-    (property "Footprint" "" (at 69.85 69.85 0)
+    (property "Footprint" "Inductor_SMD:L_0603_1608Metric_Pad1.05x0.95mm_HandSolder" (at 69.85 69.85 0)
       (effects (font (size 1.27 1.27)) hide)
     )
@@
       (effects (font (size 1.27 1.27)) (justify left))
     )
-    (property "Footprint" "" (at 227.6348 82.55 0)
+    (property "Footprint" "Capacitor_SMD:C_0603_1608Metric_Pad1.08x0.95mm_HandSolder" (at 227.6348 82.55 0)
       (effects (font (size 1.27 1.27)) hide)
     )
@@
       (effects (font (size 1.27 1.27)) (justify left))
     )
-    (property "Footprint" "" (at 199.0852 27.94 0)
+    (property "Footprint" "Capacitor_SMD:C_0603_1608Metric_Pad1.08x0.95mm_HandSolder" (at 199.0852 27.94 0)
       (effects (font (size 1.27 1.27)) hide)
     )
@@
       (effects (font (size 1.27 1.27)) (justify left))
     )
-    (property "Footprint" "" (at 253.6952 26.67 0)
+    (property "Footprint" "Capacitor_SMD:C_0603_1608Metric_Pad1.08x0.95mm_HandSolder" (at 253.6952 26.67 0)
       (effects (font (size 1.27 1.27)) hide)
     )
@@
       (effects (font (size 1.27 1.27)))
     )
-    (property "Footprint" "Button_Switch_SMD:SW_MEC_5GSH9" (at 203.2 106.68 0)
+    (property "Footprint" "Button_Switch_SMD:SW_Push_1P1T_NO_6x6mm_H9.5mm" (at 203.2 106.68 0)
       (effects (font (size 1.27 1.27)) hide)
     )
@@
     )
   )
-  (symbol (lib_id "power:GND") (at 114.3 189.23 0) (unit 1)
-    (in_bom yes) (on_board yes) (dnp no) (fields_autoplaced)
-    (property "Reference" "#PWR017" (at 114.3 195.58 0)
-      (effects (font (size 1.27 1.27)) hide)
-    )
-    (property "Value" "GND" (at 114.3 194.31 0)
-      (effects (font (size 1.27 1.27)))
-    )
-    (property "Footprint" "" (at 114.3 189.23 0)
-      (effects (font (size 1.27 1.27)) hide)
-    )
-    (property "Datasheet" "" (at 114.3 189.23 0)
+  (symbol (lib_id "power:GND") (at 116.84 190.5 0) (unit 1)
+    (in_bom yes) (on_board yes) (dnp no) (fields_autoplaced)
+    (property "Reference" "#PWR017" (at 116.84 196.85 0)
+      (effects (font (size 1.27 1.27)) hide)
+    )
+    (property "Value" "GND" (at 116.84 195.58 0)
+      (effects (font (size 1.27 1.27)))
+    )
+    (property "Footprint" "" (at 116.84 190.5 0)
+      (effects (font (size 1.27 1.27)) hide)
+    )
+    (property "Datasheet" "" (at 116.84 190.5 0)
       (effects (font (size 1.27 1.27)) hide)
     )
@@
       (effects (font (size 1.27 1.27)))
     )
-    (property "Footprint" "Resistor_SMD:R_0805_2012Metric_Pad1.20x1.40mm_HandSolder" (at 181.61 141.478 90)
+    (property "Footprint" "Resistor_SMD:R_0603_1608Metric_Pad0.98x0.95mm_HandSolder" (at 181.61 141.478 90)
       (effects (font (size 1.27 1.27)) hide)
     )
@@
       (effects (font (size 1.27 1.27)) (justify left))
     )
-    (property "Footprint" "" (at 243.5352 26.67 0)
+    (property "Footprint" "Capacitor_SMD:C_0603_1608Metric_Pad1.08x0.95mm_HandSolder" (at 243.5352 26.67 0)
       (effects (font (size 1.27 1.27)) hide)
     )
@@
       (effects (font (size 1.27 1.27)) (justify left))
     )
-    (property "Footprint" "" (at 233.3752 26.67 0)
+    (property "Footprint" "Capacitor_SMD:C_0603_1608Metric_Pad1.08x0.95mm_HandSolder" (at 233.3752 26.67 0)
       (effects (font (size 1.27 1.27)) hide)
     )
@@
       (effects (font (size 1.27 1.27)) (justify right))
     )
-    (property "Footprint" "" (at 75.2348 69.85 0)
+    (property "Footprint" "Capacitor_SMD:C_0603_1608Metric_Pad1.08x0.95mm_HandSolder" (at 75.2348 69.85 0)
       (effects (font (size 1.27 1.27)) hide)
     )
@@
       (effects (font (size 1.27 1.27)) (justify left))
     )
-    (property "Footprint" "" (at 209.2452 27.94 0)
+    (property "Footprint" "Capacitor_SMD:C_0603_1608Metric_Pad1.08x0.95mm_HandSolder" (at 209.2452 27.94 0)
       (effects (font (size 1.27 1.27)) hide)
     )
@@
       (effects (font (size 1.27 1.27)) (justify left))
     )
-    (property "Footprint" "" (at 246.6848 80.01 0)
+    (property "Footprint" "Capacitor_SMD:C_0603_1608Metric_Pad1.08x0.95mm_HandSolder" (at 246.6848 80.01 0)
       (effects (font (size 1.27 1.27)) hide)
     )
@@
       (effects (font (size 1.27 1.27)))
     )
-    (property "Footprint" "Resistor_SMD:R_0805_2012Metric_Pad1.20x1.40mm_HandSolder" (at 181.61 147.828 90)
+    (property "Footprint" "Resistor_SMD:R_0603_1608Metric_Pad0.98x0.95mm_HandSolder" (at 181.61 147.828 90)
       (effects (font (size 1.27 1.27)) hide)
     )
@@
       (effects (font (size 1.27 1.27)) (justify left))
     )
-    (property "Footprint" "" (at 169.8752 24.13 0)
+    (property "Footprint" "Capacitor_SMD:C_0603_1608Metric_Pad1.08x0.95mm_HandSolder" (at 169.8752 24.13 0)
       (effects (font (size 1.27 1.27)) hide)
     )
@@
       (effects (font (size 1.27 1.27)))
     )
-    (property "Footprint" "" (at 203.2 119.38 0)
-      (effects (font (size 1.27 1.27)) hide)
-    )
+    (property "Footprint" "Button_Switch_SMD:SW_Push_1P1T_NO_6x6mm_H9.5mm" (at 203.2 119.38 0)
+      (effects (font (size 1.27 1.27)) hide)
+    )
