File: cr2-clone/cr2-clone.kicad_sch (KiCad schematic)
At the start: 11 parts, among them J1 USB_C_Receptacle_USB2.0_16P

Commit message: added peripherals
Connections:
- net D+ renamed D_P
- net D_P: now also D1.3 (I/O2); no longer D1.2 (I/O1)
- net D- renamed D_N
- net D_N: now also D1.2 (I/O1); no longer D1.3 (I/O2)
Changed lines of the file:
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@@
   (junction (at 111.76 31.75) (diameter 0) (color 0 0 0 0)
   )
+  (junction (at 45.72 44.45) (diameter 0) (color 0 0 0 0)
+  )
   (junction (at 54.61 25.4) (diameter 0) (color 0 0 0 0)
   )
@@
   )
   (junction (at 132.08 24.13) (diameter 0) (color 0 0 0 0)
+  )
+  (junction (at 45.72 39.37) (diameter 0) (color 0 0 0 0)
   )
   (no_connect (at 99.06 29.21))
@@
     (stroke (width 0) (type default))
   )
+  (wire (pts (xy 45.72 39.37) (xy 45.72 40.64))
+    (stroke (width 0) (type default))
+  )
   (wire (pts (xy 109.22 24.13) (xy 111.76 24.13))
     (stroke (width 0) (type default))
   )
+  (wire (pts (xy 92.71 60.96) (xy 90.17 60.96))
+    (stroke (width 0) (type default))
+  )
   (wire (pts (xy 99.06 24.13) (xy 101.6 24.13))
     (stroke (width 0) (type default))
   )
+  (wire (pts (xy 46.99 44.45) (xy 45.72 44.45))
+    (stroke (width 0) (type default))
+  )
   (wire (pts (xy 99.06 26.67) (xy 105.41 26.67))
     (stroke (width 0) (type default))
@@
     (stroke (width 0) (type default))
   )
-  (wire (pts (xy 45.72 43.18) (xy 45.72 45.72))
+  (wire (pts (xy 45.72 43.18) (xy 45.72 44.45))
+    (stroke (width 0) (type default))
+  )
+  (wire (pts (xy 45.72 44.45) (xy 45.72 45.72))
     (stroke (width 0) (type default))
   )
@@
     (stroke (width 0) (type default))
   )
+  (wire (pts (xy 63.5 60.96) (xy 64.77 60.96))
+    (stroke (width 0) (type default))
+  )
   (wire (pts (xy 111.76 24.13) (xy 121.92 24.13))
     (stroke (width 0) (type default))
   )
-  (wire (pts (xy 45.72 38.1) (xy 45.72 40.64))
+  (wire (pts (xy 125.73 105.41) (xy 121.92 105.41))
+    (stroke (width 0) (type default))
+  )
+  (wire (pts (xy 46.99 39.37) (xy 45.72 39.37))
+    (stroke (width 0) (type default))
+  )
+  (wire (pts (xy 45.72 38.1) (xy 45.72 39.37))
+    (stroke (width 0) (type default))
+  )
+  (wire (pts (xy 123.19 102.87) (xy 125.73 102.87))
     (stroke (width 0) (type default))
   )
@@
     (stroke (width 0) (type default))
   )
-  (global_label "D+" (shape input) (at 64.77 60.96 180) (fields_autoplaced)
-    (effects (font (size 1.27 1.27)) (justify right))
-    (property "Intersheetrefs" "${INTERSHEET_REFS}" (at 58.9424 60.96 0)
-      (effects (font (size 1.27 1.27)) (justify right) hide)
-    )
-  )
-  (global_label "D-" (shape input) (at 45.72 39.37 0) (fields_autoplaced)
-    (effects (font (size 1.27 1.27)) (justify left))
-    (property "Intersheetrefs" "${INTERSHEET_REFS}" (at 51.5476 39.37 0)
-      (effects (font (size 1.27 1.27)) (justify left) hide)
-    )
+  (label "D_P" (at 46.99 44.45 0) (fields_autoplaced)
+    (effects (font (size 1.27 1.27)) (justify left bottom))
+  )
+  (label "D_N" (at 63.5 60.96 90) (fields_autoplaced)
+    (effects (font (size 1.27 1.27)) (justify left bottom))
+  )
+  (label "D_P" (at 121.92 105.41 180) (fields_autoplaced)
+    (effects (font (size 1.27 1.27)) (justify right bottom))
+  )
+  (label "D_N" (at 46.99 39.37 0) (fields_autoplaced)
+    (effects (font (size 1.27 1.27)) (justify left bottom))
+  )
+  (label "D_N" (at 123.19 102.87 180) (fields_autoplaced)
+    (effects (font (size 1.27 1.27)) (justify right bottom))
+  )
+  (label "D_P" (at 92.71 60.96 270) (fields_autoplaced)
+    (effects (font (size 1.27 1.27)) (justify right bottom))
   )
   (global_label "VCC" (shape input) (at 21.59 78.74 180) (fields_autoplaced)
@@
     )
   )
-  (global_label "D-" (shape input) (at 90.17 60.96 0) (fields_autoplaced)
+  (hierarchical_label "PA_SDO" (shape input) (at 154.94 109.22 180) (fields_autoplaced)
+    (effects (font (size 1.27 1.27)) (justify right))
+  )
+  (hierarchical_label "PA_MODE" (shape input) (at 154.94 132.08 180) (fields_autoplaced)
+    (effects (font (size 1.27 1.27)) (justify right))
+  )
+  (hierarchical_label "PA_PDN" (shape input) (at 154.94 120.65 180) (fields_autoplaced)
+    (effects (font (size 1.27 1.27)) (justify right))
+  )
+  (hierarchical_label "PA_ANT_SEL" (shape input) (at 154.94 129.54 180) (fields_autoplaced)
+    (effects (font (size 1.27 1.27)) (justify right))
+  )
+  (hierarchical_label "D_N" (shape bidirectional) (at 125.73 102.87 0) (fields_autoplaced)
     (effects (font (size 1.27 1.27)) (justify left))
-    (property "Intersheetrefs" "${INTERSHEET_REFS}" (at 95.9976 60.96 0)
-      (effects (font (size 1.27 1.27)) (justify left) hide)
-    )
-  )
-  (global_label "D+" (shape input) (at 45.72 44.45 0) (fields_autoplaced)
+  )
+  (hierarchical_label "D_P" (shape bidirectional) (at 125.73 105.41 0) (fields_autoplaced)
     (effects (font (size 1.27 1.27)) (justify left))
-    (property "Intersheetrefs" "${INTERSHEET_REFS}" (at 51.5476 44.45 0)
-      (effects (font (size 1.27 1.27)) (justify left) hide)
-    )
+  )
+  (hierarchical_label "TX_EN" (shape input) (at 154.94 125.73 180) (fields_autoplaced)
+    (effects (font (size 1.27 1.27)) (justify right))
+  )
+  (hierarchical_label "PA_CS" (shape input) (at 154.94 116.84 180) (fields_autoplaced)
+    (effects (font (size 1.27 1.27)) (justify right))
+  )
+  (hierarchical_label "ANT" (shape bidirectional) (at 154.94 102.87 180) (fields_autoplaced)
+    (effects (font (size 1.27 1.27)) (justify right))
+  )
+  (hierarchical_label "RX_EN" (shape input) (at 154.94 123.19 180) (fields_autoplaced)
+    (effects (font (size 1.27 1.27)) (justify right))
+  )
+  (hierarchical_label "PA_SDI" (shape output) (at 154.94 111.76 180) (fields_autoplaced)
+    (effects (font (size 1.27 1.27)) (justify right))
+  )
+  (hierarchical_label "PA_SCK" (shape input) (at 154.94 114.3 180) (fields_autoplaced)
+    (effects (font (size 1.27 1.27)) (justify right))
   )
   (symbol (lib_id "power:VCC") (at 132.08 24.13 0) (unit 1)
@@
     )
   )
-  (sheet (at 125.73 99.06) (size 52.07 53.34) (fields_autoplaced)
+  (sheet (at 125.73 99.06) (size 29.21 39.37) (fields_autoplaced)
     (stroke (width 0.1524) (type solid))
     (fill (color 0 0 0 0.0000))
@@
       (effects (font (size 1.27 1.27)) (justify left bottom))
     )
-    (property "Sheetfile" "MCU.kicad_sch" (at 125.73 152.9846 0)
+    (property "Sheetfile" "MCU.kicad_sch" (at 125.73 139.0146 0)
       (effects (font (size 1.27 1.27)) (justify left top))
     )

Commit message: added footprint, init pcb design
Parts:
- added J2, J6: Conn_01x05, Conn:SMA_EDGE, symbol Connector_Generic:Conn_01x05
- added J7: Conn_01x02_Pin, Connector_PinSocket_2.54mm:PinSocket_1x02_P2.54mm_Vertical, symbol Connector:Conn_01x02_Pin
- C1: footprint Capacitor_SMD:C_0201_0603Metric_Pad0.64x0.40mm_HandSolder -> Capacitor_SMD:C_0603_1608Metric_Pad1.08x0.95mm_HandSolder
- C2, C3, C4: footprint (none) -> Capacitor_SMD:C_0603_1608Metric_Pad1.08x0.95mm_HandSolder
- J1: footprint (none) -> Connector_USB:USB_C_Receptacle_HCTL_HC-TYPE-C-16P-01A
- L1, L2: footprint (none) -> Inductor_SMD:L_0603_1608Metric_Pad1.05x0.95mm_HandSolder
- R1, R2: footprint (none) -> Resistor_SMD:R_0603_1608Metric_Pad0.98x0.95mm_HandSolder
- U1: footprint (none) -> Package_TO_SOT_SMD:SOT-563
Connections:
- net D_N: now also J7.1 (Pin_1)
- net D_P: now also J7.2 (Pin_2)
- net GND: now also U1.1 (GND), J2.1 (Pin_1), J2.3 (Pin_3), J2.4 (Pin_4), J2.5 (Pin_5), J6.1 (Pin_1), J6.3 (Pin_3), J6.4 (Pin_4), J6.5 (Pin_5); no longer U1. (VIN)
- net at R1.2, R2.1: now also U1.5 (FB); no longer U1. (VIN)
- net at C2.1, L1.2: now also U1.3 (VIN), U1.4 (EN); no longer U1. (VIN)
- net at L2.1: now also U1.2 (SW); no longer U1. (VIN)
- new net RF_FRONT_END/ANT_1: J2.2 (Pin_2)
- new net RF_FRONT_END/ANT_2: J6.2 (Pin_2)
- no-connect marks 1 -> 6
Other:
- added sheet RF_FRONT_END (RF.kicad_sch)
- sheet MCU ports: added ANT, D_N, D_P, PA_ANT_SEL, PA_CS, PA_MODE, PA_PDN, PA_SCK, PA_SDI, PA_SDO, RX_EN, TX_EN; removed none
